File: hardware/industrial-analog-out-v2.kicad_sch (KiCad schematic)
At the start: 47 parts

Commit message: remove rescue lib stuff
Parts:
- C1, C2, C5, C7: value (none) -> 4.7µF; footprint (none) -> kicad-libraries:C0805; symbol industrial-analog-out-v2-rescue:C -> tinkerforge:C
- C10: value (none) -> 100pF; footprint (none) -> kicad-libraries:C0603F; symbol industrial-analog-out-v2-rescue:C -> tinkerforge:C
- C11: value (none) -> 1nF; footprint (none) -> kicad-libraries:C0603F; symbol industrial-analog-out-v2-rescue:C -> tinkerforge:C
- C12: value (none) -> 220pF; footprint (none) -> kicad-libraries:C0402F; symbol industrial-analog-out-v2-rescue:C -> tinkerforge:C
- C13: value (none) -> 1uF; footprint (none) -> kicad-libraries:C0603F; symbol industrial-analog-out-v2-rescue:C -> tinkerforge:C
- C14, C6, C8, C9: value (none) -> 100nF; footprint (none) -> kicad-libraries:C0603F; symbol industrial-analog-out-v2-rescue:C -> tinkerforge:C
- C3: value (none) -> 10uF; footprint (none) -> kicad-libraries:C0805; symbol industrial-analog-out-v2-rescue:C -> tinkerforge:C
- C4: value (none) -> 270pF; footprint (none) -> kicad-libraries:C0603F; symbol industrial-analog-out-v2-rescue:C -> tinkerforge:C
- D1: value (none) -> B0520LW; footprint (none) -> kicad-libraries:SOD-123; symbol industrial-analog-out-v2-rescue:DIODESCH -> tinkerforge:DIODESCH
- D2, D3: value (none) -> DESD1P0RFW; footprint (none) -> kicad-libraries:SOT23-3; symbol industrial-analog-out-v2-rescue:TVS2 -> tinkerforge:TVS2
- D4: value (none) -> CDSOD323-T15SC; footprint (none) -> kicad-libraries:SOD-323; symbol industrial-analog-out-v2-rescue:TVS -> tinkerforge:TVS
- D5, D6: value (none) -> blue; footprint (none) -> kicad-libraries:D0603F; symbol industrial-analog-out-v2-rescue:LED -> tinkerforge:LED
- F1: value (none) -> OZCJ0035FF2G; footprint (none) -> kicad-libraries:C1206; symbol industrial-analog-out-v2-rescue:FUSE -> tinkerforge:FUSE
- L1, L3, L4: value (none) -> FB; footprint (none) -> kicad-libraries:R0603F; symbol industrial-analog-out-v2-rescue:INDUCT -> tinkerforge:INDUCT
- L2: value (none) -> 10µH; footprint (none) -> kicad-libraries:NR3030; symbol industrial-analog-out-v2-rescue:INDUCTOR -> tinkerforge:INDUCTOR
- P1: value (none) -> CON-SENSOR2; footprint (none) -> kicad-libraries:CON-SENSOR2; symbol industrial-analog-out-v2-rescue:CON-SENSOR2 -> tinkerforge:CON-SENSOR2
- P2: value (none) -> CONN_8; footprint (none) -> kicad-libraries:OQ_8P; symbol industrial-analog-out-v2-rescue:CONN_8 -> tinkerforge:CONN_8
- P3: value (none) -> DEBUG; footprint (none) -> kicad-libraries:DEBUG_PAD; symbol industrial-analog-out-v2-rescue:CONN_01X01 -> tinkerforge:CONN_01X01
- P4: value (none) -> BOOT; footprint (none) -> kicad-libraries:SolderJumper; symbol industrial-analog-out-v2-rescue:CONN_01X02 -> tinkerforge:CONN_01X02
- R1: value (none) -> 1M; footprint (none) -> kicad-libraries:R0603F; symbol industrial-analog-out-v2-rescue:R -> tinkerforge:R
- R2: value (none) -> 13.3k; footprint (none) -> kicad-libraries:R0603F; symbol industrial-analog-out-v2-rescue:R -> tinkerforge:R
- R3: value (none) -> 118k; footprint (none) -> kicad-libraries:R0603F; symbol industrial-analog-out-v2-rescue:R -> tinkerforge:R
- R4: value (none) -> 10k; footprint (none) -> kicad-libraries:R0603F; symbol industrial-analog-out-v2-rescue:R -> tinkerforge:R
- R5: value (none) -> DNP; footprint (none) -> kicad-libraries:R0603F; symbol industrial-analog-out-v2-rescue:R -> tinkerforge:R
- R6, R7: value (none) -> 15; footprint (none) -> kicad-libraries:R0603F; symbol industrial-analog-out-v2-rescue:R -> tinkerforge:R
- R8: value (none) -> 10; footprint (none) -> kicad-libraries:R0603F; symbol industrial-analog-out-v2-rescue:R -> tinkerforge:R
- RP1, RP2: value (none) -> 82; footprint (none) -> kicad-libraries:4X0402; symbol industrial-analog-out-v2-rescue:R_PACK4 -> tinkerforge:R_PACK4
- RP3: value (none) -> 1k; footprint (none) -> kicad-libraries:4X0603; symbol industrial-analog-out-v2-rescue:R_PACK4 -> tinkerforge:R_PACK4
- U1: value (none) -> LMR62014X; footprint (none) -> kicad-libraries:SOT23-5; symbol industrial-analog-out-v2-rescue:LMR62014X -> tinkerforge:LMR62014X
- U2: value (none) -> XMC1100; footprint (none) -> kicad-libraries:QFN24-4x4mm-0.5mm; symbol industrial-analog-out-v2-rescue:XMC1XXX24 -> tinkerforge:XMC1XXX24
- U3: value (none) -> DACX760; footprint (none) -> kicad-libraries:TSSOP24-44-PWR; symbol industrial-analog-out-v2-rescue:DACX760 -> tinkerforge:DACX760
- U4, U5, U6, U7: value (none) -> DRILL; footprint (none) -> kicad-libraries:DRILL_NP; symbol industrial-analog-out-v2-rescue:DRILL -> tinkerforge:DRILL
Connections:
- net M-CLK: now also RP2.2 (P2), U3.8 (SCLK)
- net M-CS: now also RP2.1 (P1), U3.7 (LATCH)
- net M-MISO: now also RP2.3 (P3), U3.10 (SDO)
- net M-MOSI: now also RP2.4 (P4), U3.9 (SDIN)
- net P0.2: now also RP2.5 (R4), U2.1 (P2.0_AIO)
- net S-CLK: now also RP1.7 (R2), U2.11 (P1.3_IHO)
- net S-CS: now also RP1.8 (R1), U2.20 (P0.9_IO)
- net S-MISO: now also RP1.5 (R4), U2.18 (P0.7_IO)
- net S-MOSI: now also RP1.6 (R3), U2.12 (P1.2_IHO)
- new net: F1.2, P2.1, P2.3
- new net: L4.1, P2.5
- new net: P2.7, R8.1
- new net: R5.1, U3.13 (ISET-R)
- new net: C8.1, U3.14 (REFOUT), U3.15 (REFIN)
- new net: C11.2, U3.17 (CMP)
- new net: R8.2, U3.19 (IOUT)
- new net: C11.1, R7.2, U3.21 (VOUT)
- new net: R6.2, U3.22 (+VSENSE)
- new net: R4.2, U3.3 (nALARM)
- new net: L4.2, R6.1, R7.1
- new net: D1.1 (A), L2.1, U1.1 (SW)
- new net: C4.2, R2.1, R3.2, U1.3 (FB)
- new net: R1.2, U1.4 (nSHDN)
- new net: C2.2, L1.1, L2.2, U1.5 (VIN)
- new net: C4.1, C5.2, D1.2 (K), L3.2
- new net: P1.4, RP1.1 (P1)
- new net: P1.5, RP1.2 (P2)
- new net: P1.6, RP1.3 (P3)
- new net: C12.1, P1.7, RP1.4 (P4)
- new net: P3.1 (P1), U2.15 (P0.0_IO)
- new net: RP2.8 (R1), U2.22 (P0.13_IO)
- new net: RP2.7 (R2), U2.23 (P0.14_IO)
- new net: RP2.6 (R3), U2.24 (P0.15_IO)
- new net: RP3.5 (R4), U2.13 (P1.1_IHO)
- new net: RP3.8 (R1), U2.14 (P1.0_IHO)
- new net: P4.2 (P2), U2.7 (P2.10_AIO)
- new net: D5.2 (K), RP3.1 (P1)
- new net: D6.2 (K), RP3.4 (P4)
- new net +5V: C1.2, L1.2, P1.1
- new net 12V: C10.2, C7.2, C9.2, D2.2 (K), D3.2 (K), F1.1, L3.1, U3.24 (AVDD)
- new net 3V3: C13.1, C14.1, C3.1, D5.1 (A), D6.1 (A), P1.3, R4.1, U2.10 (VDDP/VDD), U3.2 (DVDD)
- new net GND: C1.1, C10.1, C12.2, C13.2, C14.2, C2.1, C3.2, C5.1, C6.2, C7.1, C8.2, C9.1, D2.1 (A), D3.1 (A), D4.2 (K), P1.2, P1.EP, P2.2, P2.4, P2.6, P2.8, P4.1 (P1), R2.2, R5.2, U1.2 (GND), U2.9 (VSSP/VSS), U2.EXP (VSSP), U3.1 (AVSS), U3.11 (GND), U3.12 (GND), U3.16 (DVDD-EN), U3.23 (-VSENSE), U3.4 (GND), U3.5 (CLR-SEL), U3.6 (CLR)

Commit message: Data Cleanup
Other:
- note added: "Copyright Tinkerforge GmbH 2023. This documentation describes Open Hardware and is licensed under the CERN OHL v. 1.1. You may redistribute and modify this documentation under the terms of the CERN OHL v.1.1. (http://ohwr.org/cernohl). This documentation is distributed WITHOUT ANY EXPRESS OR IMPLIED WARRANTY, INCLUDING OF MERCHANTABILITY, SATISFACTORY QUALITY AND FITNESS FOR A PARTICULAR PURPOSE.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"
- note removed: "Copyright Tinkerforge GmbH 2018. This documentation describes Open Hardware and is licensed under the CERN OHL v. 1.1. You may redistribute and modify this documentation under the terms of the CERN OHL v.1.1. (http://ohwr.org/cernohl). This documentation is distributed WITHOUT ANY EXPRESS OR IMPLIED WARRANTY, INCLUDING OF MERCHANTABILITY, SATISFACTORY QUALITY AND FITNESS FOR A PARTICULAR PURPOSE.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"
